File: SuperHAT V2.kicad_pcb (KiCad board)
At the start: 4 copper layers, 65 x 56.5 mm, 82 parts, among them J1 GPIO, J10 Qwiic_RA, J11 Conn_01x02, J12 B02B-PASK-1, J2 Conn_01x03, J4 Conn_01x03, J5 Qwiic_RA, J6 Qwiic_Vertical, J7 Qwiic_Vertical, J8 SM04B-GHS-TB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

Commit message: Organized version.
Changed lines of the file:
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@@
 		(grid_origin 100 100)
 		(pcbplotparams
-			(layerselection 0x00010fc_ffffffff)
+			(layerselection 0x000100c_7ffffff8)
 			(plot_on_all_layers_selection 0x0000000_00000000)
 			(disableapertmacros no)
-			(usegerberextensions yes)
+			(usegerberextensions no)
 			(usegerberattributes no)
 			(usegerberadvancedattributes no)
@@
 			(plotinvisibletext no)
 			(sketchpadsonfab no)
-			(subtractmaskfromsilk yes)
+			(subtractmaskfromsilk no)
 			(outputformat 1)
 			(mirror no)
 			(drillshape 0)
 			(scaleselection 1)
-			(outputdirectory "../KiCAD Exports/SuperHAT/")
+			(outputdirectory "C:/KiCAD/KiCAD Exports/SuperHAT/")
 		)
 	)
@@
 		(tags "SparkFun")
 		(property "Reference" "J7"
-			(at -0.301 -0.445 360)
+			(at -0.301 -0.445 0)
 			(layer "F.SilkS")
 			(effects
@@
 		(at 107.210002 98.249999)
 		(property "Reference" "R14"
-			(at 2.25 0 270)
+			(at 2.25 0 -90)
 			(unlocked yes)
 			(layer "F.SilkS")
@@
 		(tags "CHP0805AFX-2200ELF ")
 		(property "Reference" "R13"
-			(at -2.1 -0.000001 270)
+			(at -2.1 -0.000001 -90)
 			(unlocked yes)
 			(layer "F.SilkS")
