File: SuperHAT V2.kicad_sch (KiCad schematic)
At the start: 80 parts, among them J1 GPIO, J10 Qwiic_RA, J11 Conn_01x02, J12 B02B-PASK-1, J2 Conn_01x03, J4 Conn_01x03, J5 Qwiic_RA, J6 Qwiic_Vertical, J7 Qwiic_Vertical, J8 SM04B-GHS-TB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

Commit message: Organized version.
Parts:
- J3: value ~ -> MR30PW-M
Connections:
- net at U4.6 (OUT1): now also J12.1; no longer J12.2
- net at U4.8 (OUT2): now also J12.2; no longer J12.1
Other:
- note added: "5V Output"
- note added: "Current Sensor"
- note added: "DC Motor Driver"
- note added: "GPIO Pins"
- note added: "I2C Connectors"
- note added: "MOSFET Switching Circuits"
- note added: "Power Indicators"
- note added: "Power Input"
- note added: "Pull-up Resistor Arrays"
- note added: "Servos"
- note added: "Stepper Motor Driver"
- note added: "eFuse for Pi"
- title: SuperHAT (SHAT) -> SuperHAT
- moved on the sheet: C1, C10, C11, C12, C2, C3, C4, C5, C6, C7, C8, C9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
